File: board/IAS3A.kicad_pcb (KiCad board)
At the start: 2 copper layers, 46 x 28 mm, 14 parts, among them J1 Address, J2 Flow Ext, J3 Pressure Ext, J4 Pressure Int, U1 STM32F030F4Px, X1 I2C-6P, X2 SWD

Commit message: WIP
Routing:
- net +5V: track 0.00 -> 55.3 mm, vias 0 -> 1
- net +3V3: track 0.00 -> 46.0 mm, vias 0 -> 2
- net Net-(J4-Pad2): track 0.00 -> 42.9 mm
- net GND: track 0.00 -> 22.2 mm, vias 0 -> 5
- net /ALERT: track 0.00 -> 21.9 mm, vias 0 -> 2
- net Net-(J3-Pad2): track 0.00 -> 20.1 mm
- net /SDA: track 0.00 -> 18.6 mm, vias 0 -> 2
- net Net-(R1-Pad2): track 0.00 -> 16.6 mm, vias 0 -> 2
- net Net-(J1-Pad2): track 0.00 -> 15.6 mm, vias 0 -> 2
- net Net-(J2-Pad2): track 0.00 -> 15.4 mm
- net /SCL: track 0.00 -> 12.4 mm, vias 0 -> 2
- net Net-(C1-Pad1): track 0.00 -> 9.10 mm, vias 0 -> 2
- net /SWDIO: track 0.00 -> 7.03 mm
- net Net-(R3-Pad2): track 0.00 -> 5.58 mm
- net /SWCLK: track 0.00 -> 3.24 mm
- added copper zone on B.Cu, net GND
Other:
- net class Default: trace_width 0.25 -> 0.4
- net class PWR added: clearance 0.2, trace_width 0.6, via_dia 0.9, via_drill 0.6
- board text added: "COLD"
- board text added: "IAS3A v1.0"
- board text removed: "CLD"
